File: transmitter/transmitter.kicad_pcb (KiCad board)
At the start: 2 copper layers, 8 parts, among them J1 Conn_01x05, J2 Conn_01x05, U1 NRF24L01_Breakout, U2 AMS1117-3.3

Commit message: Completed transmitter PCB and rough BOM, updated journal
Parts:
- added S1: FlashLightToggle, Button_Switch_THT:SW_Slide_SPDT_Straight_CK_OS102011MS2Q, F.Cu at (210.0, 69.3)
- added S2: OnOff, Button_Switch_THT:SW_Slide_SPDT_Straight_CK_OS102011MS2Q, F.Cu at (133.9, 69.0)
- BT1: footprint Connector_JST:JST_XH_B3B-XH-A_1x03_P2.50mm_Vertical -> Connector_PinHeader_2.54mm:PinHeader_1x02_P2.54mm_Vertical; moved to B.Cu
- moved U2 43.1 mm to (198.0, 63.0)
- moved C1 31.6 mm to (157.0, 62.0)
- moved J1 28.8 mm to (152.0, 85.5)
- moved BT1 25.0 mm to (155.0, 71.0), turned to 90 degrees
- moved A1 23.8 mm to (165.8, 76.3)
- moved C2 22.4 mm to (183.6, 62.0)
- moved U1 21.0 mm to (167.4, 66.5), turned to 90 degrees
- moved J2 3.12 mm to (196.0, 85.5)
Routing:
- net GND: track 0.00 -> 193.8 mm, vias 0 -> 1
- net Net-(U2-VI): track 0.00 -> 82.6 mm
- net +5V: track 0.00 -> 77.1 mm
- net Net-(A1-D10): track 0.00 -> 56.9 mm, vias 0 -> 1
- net Net-(A1-D2): track 0.00 -> 53.6 mm
- net Net-(A1-SCK): track 0.00 -> 51.0 mm, vias 0 -> 2
- net Net-(A1-MOSI): track 0.00 -> 50.8 mm, vias 0 -> 1
- net Net-(A1-MISO): track 0.00 -> 50.5 mm, vias 0 -> 1
- net X1: track 0.00 -> 42.5 mm
- net Net-(A1-D9): track 0.00 -> 41.2 mm, vias 0 -> 1
- net +3.3V: track 0.00 -> 38.3 mm, vias 0 -> 1
- net Y1: track 0.00 -> 31.5 mm
- net X2: track 0.00 -> 26.8 mm
- net Net-(BT1-+): track 0.00 -> 24.4 mm
- net Y2: track 0.00 -> 16.5 mm
Other:
- board outline added: 122 x 77 mm
- board text added: "Joystick Left"
- board text added: "Joystick Right"

Commit message: Updated BOM, total time spent
Parts:
- C1, C2: value 10mF -> 10uF
Routing:
- net Net-(U2-VI): track 82.6 -> 73.2 mm
Other:
- outline, holes or cut-outs redrawn
Changed lines of the file:
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@@
 			)
 		)
-		(property "Value" "10mF"
+		(property "Value" "10uF"
 			(at 2.5 5.25 0)
 			(layer "F.Fab")
@@
 		(tags "CMS SOT")
 		(property "Reference" "U2"
-			(at 0 -4.5 0)
+			(at -2 -4.5 0)
 			(layer "F.SilkS")
 			(effects
@@
 		)
 		(property "Value" "OnOff"
-			(at 2 4 0)
+			(at 0.1 -5 0)
 			(layer "F.Fab")
 			(effects
@@
 		)
 		(property "Value" "FlashLightToggle"
-			(at 2 3.7025 0)
+			(at 2 -5.2975 0)
 			(layer "F.Fab")
 			(effects
@@
 			)
 		)
-		(property "Value" "10mF"
+		(property "Value" "10uF"
 			(at 2.5 5.25 0)
 			(layer "F.Fab")
@@
 	)
 	(gr_line
-		(start 219 51)
-		(end 184 51)
+		(start 184 51)
+		(end 202 51)
 		(stroke
 			(width 0.05)
@@
 	)
 	(gr_line
-		(start 160 51)
+		(start 144 51)
 		(end 162 51)
 		(stroke
@@
 	)
 	(gr_line
-		(start 124 59)
-		(end 130 51)
+		(start 183 116)
+		(end 234 116)
 		(stroke
 			(width 0.05)
@@
 	)
 	(gr_line
-		(start 183 116)
-		(end 234 116)
+		(start 165 39)
+		(end 181 39)
 		(stroke
 			(width 0.05)
@@
 	)
 	(gr_line
-		(start 165 39)
-		(end 181 39)
+		(start 202 51)
+		(end 235 72)
 		(stroke
 			(width 0.05)
@@
 		(layer "Edge.Cuts")
 	)
-	(gr_line
-		(start 224 58)
-		(end 219 51)
+	(gr_circle
+		(center 148 56)
+		(end 150 55)
 		(stroke
 			(width 0.05)
 			(type default)
 		)
+		(fill no)
 		(layer "Edge.Cuts")
 	)
@@
 		(layer "Edge.Cuts")
 	)
-	(gr_line
-		(start 124 59)
-		(end 113 73)
-		(stroke
-			(width 0.05)
-			(type default)
-		)
-		(layer "Edge.Cuts")
-	)
-	(gr_line
-		(start 130 51)
-		(end 160 51)
-		(stroke
-			(width 0.05)
-			(type default)
-		)
-		(layer "Edge.Cuts")
-	)
 	(gr_arc
 		(start 235 115)
@@
 		(layer "Edge.Cuts")
 	)
-	(gr_line
-		(start 224 58)
-		(end 235 72)
+	(gr_arc
+		(start 114 116)
+		(mid 113.292893 115.707107)
+		(end 113 115)
 		(stroke
 			(width 0.05)
@@
 		(layer "Edge.Cuts")
 	)
-	(gr_arc
-		(start 114 116)
-		(mid 113.292893 115.707107)
-		(end 113 115)
+	(gr_circle
+		(center 199 56)
+		(end 201 55)
 		(stroke
 			(width 0.05)
 			(type default)
 		)
+		(fill no)
 		(layer "Edge.Cuts")
 	)
@@
 	)
 	(gr_line
-		(start 113 118)
-		(end 113 118)
+		(start 113 73)
+		(end 144 51)
 		(stroke
 			(width 0.05)
@@
 	)
 	(segment
-		(start 178.5671 71)
-		(end 189.15 71)
+		(start 156.11384 61)
+		(end 140 61)
 		(width 0.2)
 		(layer "F.Cu")
@@
 	)
 	(segment
-		(start 161 56)
-		(end 141 56)
+		(start 161 61)
+		(end 162 62)
 		(width 0.2)
 		(layer "F.Cu")
@@
 	)
 	(segment
-		(start 168.401 71.401)
-		(end 178.1661 71.401)
+		(start 157.88616 61)
+		(end 157.78516 60.899)
 		(width 0.2)
 		(layer "F.Cu")
@@
 	)
 	(segment
-		(start 162 57)
-		(end 161 56)
+		(start 178.5671 71)
+		(end 189.15 71)
+		(width 0.2)
+		(layer "F.Cu")
+		(net 31)
+	)
+	(segment
+		(start 168.401 71.401)
+		(end 178.1661 71.401)
 		(width 0.2)
 		(layer "F.Cu")
@@
 	)
 	(segment
-		(start 162 62)
-		(end 162 57)
+		(start 161 61)
+		(end 157.88616 61)
 		(width 0.2)
 		(layer "F.Cu")
@@
 	)
 	(segment
-		(start 135.9 61.1)
-		(end 135.9 69)
+		(start 156.21484 60.899)
+		(end 156.11384 61)
+		(width 0.2)
+		(layer "F.Cu")
+		(net 31)
+	)
+	(segment
+		(start 157.78516 60.899)
+		(end 156.21484 60.899)
 		(width 0.2)
 		(layer "F.Cu")
@@
 	)
 	(segment
-		(start 141 56)
-		(end 135.9 61.1)
+		(start 135.9 65.1)
+		(end 135.9 69)
 		(width 0.2)
 		(layer "F.Cu")
@@
 		(width 0.2)
 		(layer "F.Cu")
+		(net 31)
+	)
+	(segment
+		(start 140 61)
+		(end 135.9 65.1)
+		(width 0.2)
+		(layer "F.Cu")
